File: KiCad/PerpetualADSR.kicad_pcb (KiCad board)
At the start: 2 copper layers, 40 x 110 mm, 38 parts, among them J1 TEST_CONN, J2 GATE, J3 CLOCK, J4 PWR_Conn, J5 OUT, SW1 EXP/LIN, U1 ATmega328P-PU, U2 MCP4921, U3 MCP3208, Y1 16MHz

Commit message: started PCB
Parts:
- removed C1, C3, C5: 0.1u, Capacitor_THT:C_Disc_D5.0mm_W2.5mm_P5.00mm
- removed C2: 4.7u, Capacitor_THT:C_Disc_D5.0mm_W2.5mm_P2.50mm
- removed C4: 10u, Capacitor_THT:C_Disc_D5.0mm_W2.5mm_P5.00mm
- removed C6: 1u, Capacitor_THT:C_Disc_D5.0mm_W2.5mm_P2.50mm
- removed C7, C8: 22p, Capacitor_THT:C_Disc_D5.0mm_W2.5mm_P5.00mm
- removed D5: GREEN, LED_THT:LED_D5.0mm
- removed D6: 5.1V, Diode_THT:D_DO-35_SOD27_P7.62mm_Horizontal
- removed D7: RED, LED_THT:LED_D5.0mm
- removed J1: TEST_CONN, Connector_PinHeader_2.54mm:PinHeader_2x06_P2.54mm_Vertical
- removed J2: GATE, PerpetualADSR:PJ301M
- removed J3: CLOCK, PerpetualADSR:PJ301M
- removed R4: 220, Resistor_THT:R_Axial_DIN0207_L6.3mm_D2.5mm_P7.62mm_Horizontal
- removed R5: 10k, Resistor_THT:R_Axial_DIN0207_L6.3mm_D2.5mm_P7.62mm_Horizontal
- removed SW1: EXP/LIN, PerpetualADSR:SLIDE_SW_OS102011MS2QN1
- removed U1: ATmega328P-PU, Package_DIP:DIP-28_W7.62mm
- removed U2: MCP4921, Package_DIP:DIP-8_W7.62mm
- removed U3: MCP3208, Package_DIP:DIP-16_W7.62mm
- removed Y1: 16MHz, Crystal:Crystal_HC49-4H_Vertical
- added CLOCK: CLOCK, PerpetualADSR:PJ301M, F.Cu at (27.0, 109.7)
- added GATE: GATE, PerpetualADSR:PJ301M, F.Cu at (17.6, 109.7)
- added OUT: OUT, PerpetualADSR:PJ301M, F.Cu at (36.4, 109.7)
- D1: value Schottky -> S
- D2: value 5.1V -> Schottky; footprint Diode_THT:D_DO-35_SOD27_P7.62mm_Horizontal -> Diode_THT:D_DO-34_SOD68_P7.62mm_Horizontal
- D3: value S -> 5.1V; footprint Diode_THT:D_DO-34_SOD68_P7.62mm_Horizontal -> Diode_THT:D_DO-35_SOD27_P7.62mm_Horizontal
- D4: value BLUE -> 5.1V; footprint LED_THT:LED_D5.0mm -> Diode_THT:D_DO-35_SOD27_P7.62mm_Horizontal
- J4: value PWR_Conn -> Conn_02x04_Counter_Clockwise; footprint Connector_IDC:IDC-Header_2x08_P2.54mm_Vertical -> Connector_PinSocket_2.54mm:PinSocket_2x04_P2.54mm_Vertical
- J5: value OUT -> Conn_02x04_Counter_Clockwise; footprint PerpetualADSR:PJ301M -> Connector_PinSocket_2.54mm:PinSocket_2x04_P2.54mm_Vertical; moved to B.Cu
- R1: value 100k -> 10k
- R2: value 1M -> 100k
- RV1: value MAX_V -> REL_T
- RV2: value ATT_T -> MAX_V
- RV3: value REL_T -> RISE_T
- RV4: value ATT_V -> RISE_V
- RV5: value FALL_V -> FALL_T
- RV6: value RISE_T -> FALL_V
- RV7: value FALL_T -> ATT_T
- RV8: value RISE_V -> ATT_V
- moved D4 79.9 mm to (20.9, 91.3)
- moved RV2 51.4 mm to (37.1, 74.5)
- moved R3 43.1 mm to (32.8, 87.5), turned to 90 degrees
- moved J5 42.9 mm to (36.5, 79.0), turned to 180 degrees
- moved RV4 41.0 mm to (21.9, 58.5)
- moved R1 35.6 mm to (40.8, 90.6), turned to 180 degrees
- moved RV8 29.6 mm to (37.1, 26.5)
- moved D2 25.1 mm to (20.8, 94.5), turned to 180 degrees
- moved J4 24.9 mm to (15.0, 79.0), turned to 180 degrees
- moved RV1 24.0 mm to (21.9, 74.5)
- moved RV5 23.7 mm to (21.9, 42.5)
- moved RV6 18.4 mm to (37.1, 42.5)
- moved D3 18.3 mm to (33.1, 94.1), turned to 0 degrees
- moved RV3 17.7 mm to (37.1, 58.5)
- moved D1 17.5 mm to (28.5, 94.5), turned to 90 degrees
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Connections:
- D1 pad 1: GATE_IN -> CLK
- D2 pad 1: GATE_IN -> GATE
- D3 pad 1: CLK_IN -> CLK
- D4 pad 1: Net-(D4-Pad1) -> GATE
- D4 pad 2: Net-(D4-Pad2) -> GND
- J4 pad 1: Net-(J4-Pad1) -> ATT_T
- J4 pad 2: Net-(J4-Pad2) -> FALL_T
- J4 pad 3: GND -> RISE_T
- J4 pad 4: GND -> REL_T
- J4 pad 6: GND -> CLK
- J4 pad 7: GND -> GATE
- J4 pad 8: GND -> +5V
- R2 pad 1: Net-(C7-Pad2) -> GND
- R3 pad 1: GND -> Net-(J2-PadTN)
- R3 pad 2: Net-(J3-PadTN) -> +5V
- RV1 pad 2: Net-(RV1-Pad2) -> REL_T
- RV2 pad 2: Net-(RV2-Pad2) -> MAX_V
- RV3 pad 2: Net-(RV3-Pad2) -> RISE_T
- RV4 pad 2: Net-(RV4-Pad2) -> RISE_V
- RV5 pad 2: Net-(RV5-Pad2) -> FALL_T
- RV6 pad 2: Net-(RV6-Pad2) -> FALL_V
- RV7 pad 2: Net-(RV7-Pad2) -> ATT_T
- RV8 pad 2: Net-(RV8-Pad2) -> ATT_V
Routing:
- added copper zone on F.Cu, net +5V
- added copper zone on B.Cu, net GND
Other:
- board size 40 x 110 mm -> 30 x 100 mm
